Commit message: create controller and firmware

File: alphabot_description/urdf/alphabot_ros2_control.xacro (robot description, xacro)
@@ -1,9 +1,22 @@
 <?xml version="1.0" encoding="UTF-8"?>
 <robot xmlns:xacro="http://www.ros.org/wiki/xacro" name="alphabot">
-    <xacro:if value="$(arg is_sim)">
-        <ros2_control type="system" name="RobotSystem">
+    <ros2_control type="system" name="RobotSystem">
+        <xacro:if value="$(arg is_sim)">
             <hardware>
                 <plugin>gazebo_ros2_control/GazeboSystem</plugin>
             </hardware>
+        </xacro:if>
+        <xacro:unless value="$(arg is_sim)">
+                <hardware>
+                    <plugin>alphabot_firmware/AlphabotInterface</plugin>
+                    <param name="left_wheel_name">wheel_right_joint</param>
+                    <param name="right_wheel_name">wheel_left_joint</param>
+                    <param name="loop_rate">30</param>
+                    <param name="usb_port">/dev/ttyCOM0</param>
+                    <param name="baud_rate">57600</param>
+                    <param name="timeout">1000</param>
+                    <param name="enc_counts_per_rev">200</param>
+                </hardware>
+            </xacro:unless>
             <joint name="wheel_right_joint">
                 <command_interface name="velocity">
@@ -23,34 +36,3 @@
             </joint>
         </ros2_control>
-    </xacro:if>
-    <!-- <xacro:unless value="$(arg is_sim)">
-        <ros2_control type="system" name="RealRobot">
-            <hardware>
-                <plugin>basebot_firmware/BasebotInterface</plugin>
-                <param name="left_wheel_name">wheel_right_joint</param>
-                <param name="right_wheel_name">wheel_left_joint</param>
-                <param name="loop_rate">30</param>
-                <param name="usb_port">/dev/ttyCOM0</param>
-                <param name="baud_rate">57600</param>
-                <param name="timeout">1000</param>
-                <param name="enc_counts_per_rev">200</param>
-            </hardware>
-            <joint name="wheel_right_joint">
-                <command_interface name="velocity">
-                    <param name= "min"> -1 </param>
-                    <param name= "max"> 1 </param>
-                </command_interface>
-                <state_interface name="velocity"/>
-                <state_interface name="position"/>
-            </joint>
-            <joint name="wheel_left_joint">
-                <command_interface name="velocity">
-                    <param name= "min"> -1 </param>
-                    <param name= "max"> 1 </param>
-                </command_interface>
-                <state_interface name="velocity"/>
-                <state_interface name="position"/>
-            </joint>
-        </ros2_control>
-    </xacro:unless> -->
 </robot>

Commit message: connection doen seccussfully

File: alphabot_description/urdf/alphabot_ros2_control.xacro (robot description, xacro)
@@ -1,5 +1,6 @@
-<?xml version="1.0" encoding="UTF-8"?>
-<robot xmlns:xacro="http://www.ros.org/wiki/xacro" name="alphabot">
-    <ros2_control type="system" name="RobotSystem">
+<?xml version="1.0"?>
+<robot xmlns:xacro="http://www.ros.org/wiki/xacro" name="bumperbot">
+    <ros2_control name="RobotSystem" type="system">
+        <!-- ros2_control Gazebo -->
         <xacro:if value="$(arg is_sim)">
             <hardware>
@@ -7,32 +8,28 @@
             </hardware>
         </xacro:if>
+        <!-- ros2_control Real Robot -->
         <xacro:unless value="$(arg is_sim)">
-                <hardware>
-                    <plugin>alphabot_firmware/AlphabotInterface</plugin>
-                    <param name="left_wheel_name">wheel_right_joint</param>
-                    <param name="right_wheel_name">wheel_left_joint</param>
-                    <param name="loop_rate">30</param>
-                    <param name="usb_port">/dev/ttyCOM0</param>
-                    <param name="baud_rate">57600</param>
-                    <param name="timeout">1000</param>
-                    <param name="enc_counts_per_rev">200</param>
-                </hardware>
-            </xacro:unless>
-            <joint name="wheel_right_joint">
-                <command_interface name="velocity">
-                    <param name= "min"> -1 </param>
-                    <param name= "max"> 1 </param>
-                </command_interface>
-                <state_interface name="velocity"/>
-                <state_interface name="position"/>
-            </joint>
-            <joint name="wheel_left_joint">
-                <command_interface name="velocity">
-                    <param name= "min"> -1 </param>
-                    <param name= "max"> 1 </param>
-                </command_interface>
-                <state_interface name="velocity"/>
-                <state_interface name="position"/>
-            </joint>
-        </ros2_control>
+            <hardware>
+                <plugin>alphabot_firmware/AlphabotInterface</plugin>
+                <param name="port">/dev/ttyACM1</param>
+            </hardware>
+        </xacro:unless>
+        <!-- ros2_control Common Interfaces -->
+        <joint name="wheel_right_joint">
+            <command_interface name="velocity">
+              <param name="min">-1</param>
+              <param name="max">1</param>
+            </command_interface>
+            <state_interface name="position" />
+            <state_interface name="velocity" />
+        </joint>
+        <joint name="wheel_left_joint">
+            <command_interface name="velocity">
+              <param name="min">-1</param>
+              <param name="max">1</param>
+            </command_interface>
+            <state_interface name="position" />
+            <state_interface name="velocity" />
+        </joint>
+    </ros2_control>
 </robot>
