Commit message: update parameters and serial comminication style remove mpu6050 package

File: alphabot_description/urdf/camera.xacro (robot description, xacro)
@@ -1,4 +1,7 @@
 <?xml version="1.0"?>
 <robot xmlns:xacro="http://www.ros.org/wiki/xacro" >
+    <material name="red">
+        <color rgba="1 0 0 1"/>
+    </material>
     <joint name="camera_joint" type="fixed">
         <parent link="base_link"/>
