Commit message: Fixing the gazebo sim launch

File: alphabot_description/urdf/alphabot_gazebo.xacro (robot description, xacro)
@@ -1,18 +1,4 @@
 <?xml version="1.0" encoding="UTF-8"?>
 <robot xmlns:xacro="http://www.ros.org/wiki/xacro" name="alphabot">
-    <transmission name="wheel_right_transmission">
-        <plugin>transmission_interface/SimpleTransmission</plugin>
-        <actuator name="wheel_right_motor" role="actuator_right"/>
-        <joint name="wheel_right_joint"    role="joint_right">
-          <mechanical_reduction>1.0</mechanical_reduction>
-        </joint>
-      </transmission>
-      <transmission name="wheel_left_transmission">
-        <plugin>transmission_interface/SimpleTransmission</plugin>
-        <actuator name="wheel_left_motor" role="actuator_left"/>
-        <joint name="wheel_left_joint"    role="joint_left">
-          <mechanical_reduction>1.0</mechanical_reduction>
-        </joint>
-      </transmission>
     <gazebo reference="wheel_right_link">
         <mu1>100000000000000.0</mu1>
@@ -49,15 +35,6 @@
         <maxVel>0.1</maxVel>
     </gazebo>
+    <!-- ROS 2 Control -->
     <gazebo>
-    <!-- ROS 2 Humble -->
-    <xacro:if value="$(arg is_ignition)">
-      <plugin filename="ign_ros2_control-system" name="ign_ros2_control::IgnitionROS2ControlPlugin">
-        <parameters>$(find alphabot_controller)/config/alphabot_controllers.yaml</parameters>
-      </plugin>
-      <plugin filename="ignition-gazebo-imu-system" name="ignition::gazebo::systems::Imu">
-      </plugin>
-    </xacro:if>
-    <!-- ROS 2 Iron or above -->
-    <xacro:unless value="$(arg is_ignition)">
       <plugin filename="gz_ros2_control-system" name="gz_ros2_control::GazeboSimROS2ControlPlugin">
         <parameters>$(find alphabot_controller)/config/alphabot_controllers.yaml</parameters>
@@ -65,5 +42,4 @@
       <plugin filename="gz-sim-imu-system" name="gz::sim::systems::Imu">
       </plugin>
-    </xacro:unless>
   </gazebo>
 <!--

File: alphabot_description/urdf/alphabot_ros2_control.xacro (robot description, xacro)
@@ -5,5 +5,5 @@
         <xacro:if value="$(arg is_sim)">
             <hardware>
-                <plugin>gazebo_ros2_control/GazeboSystem</plugin>
+                <plugin>gz_ros2_control/GazeboSimSystem</plugin>
             </hardware>
         </xacro:if>

Commit message: fixed urdf file

File: alphabot_description/urdf/alphabot_gazebo.xacro (robot description, xacro)
@@ -2,30 +2,22 @@
 <robot xmlns:xacro="http://www.ros.org/wiki/xacro" name="alphabot">
     <gazebo reference="wheel_right_link">
-        <mu1>100000000000000.0</mu1>
-        <mu2>100000000000000.0</mu2>
-        <kp>1000000000000.0</kp>
-        <kd>10.0</kd>
-        <minDepth>0.001</minDepth>
-        <maxVel>0.1</maxVel>
-        <fdirl>1 0 0</fdirl>
+      <mu1>0.8</mu1>
+      <mu2>0.8</mu2>
+      <kp>100000.0</kp>
+      <kd>1.0</kd>
+      <minDepth>0.001</minDepth>
+      <maxVel>0.2</maxVel>
+      <fdir1>1 0 0</fdir1>
     </gazebo>
     <gazebo reference="wheel_left_link">
-        <mu1>100000000000000.0</mu1>
-        <mu2>100000000000000.0</mu2>
-        <kp>1000000000000.0</kp>
-        <kd>10.0</kd>
-        <minDepth>0.001</minDepth>
-        <maxVel>0.1</maxVel>
-        <fdirl>1 0 0</fdirl>
+      <mu1>0.8</mu1>
+      <mu2>0.8</mu2>
+      <kp>100000.0</kp>
+      <kd>1.0</kd>
+      <minDepth>0.001</minDepth>
+      <maxVel>0.2</maxVel>
+      <fdir1>1 0 0</fdir1>
     </gazebo>
-    <gazebo reference="caster_front_link">
-        <mu1>0.1</mu1>
-        <mu2>0.1</mu2>
-        <kp>1000000.0</kp>
-        <kd>100.0</kd>
-        <minDepth>0.001</minDepth>
-        <maxVel>0.1</maxVel>
-    </gazebo>
-    <gazebo reference="caster_rear_link">
+    <gazebo reference="caster_wheel">
         <mu1>0.1</mu1>
         <mu2>0.1</mu2>

File: alphabot_description/urdf/alphabot_old.urdf.xacro (robot description, xacro)
@@ -8,4 +8,10 @@
     <xacro:include filename="$(find alphabot_description)/urdf/alphabot_ros2_control.xacro"/>
     <!-- <xacro:include filename="$(find alphabot_description)/urdf/depth_camera.xacro" /> -->
+    <xacro:property name="wheel_radius" value="0.051" />
+    <xacro:property name="wheel_width" value="0.040" />
+    <xacro:property name="robot_height" value="0.093" />
+    <xacro:property name="robot_width" value="0.20" />
+    <xacro:property name="wheel_depth" value="0.22" />
+    <xacro:property name="caster_wheel" value="0.018" />
     <material name="white">
         <color rgba="1 1 1 1"/>
@@ -23,21 +29,18 @@
     <link name="base_link">
         <inertial>
-            <mass value="1.0"/>
-            <origin xyz="0 0 0"/>
-            <inertia ixx="0.002" ixy="0" ixz="0"
-                    iyy="0.002" iyz="0"
-                    izz="0.002"/>
-        </inertial>
-        <visual>
-            <origin xyz="0.0 0.0 0.066" rpy="0.0 0.0 0.0"/>
-            <geometry>
-                <box size="0.256 0.180 0.132" />
+            <mass value="2.0"/>
+            <inertia ixx="0.1" ixy="0.0" ixz="0.0" iyy="0.1" iyz="0.0" izz="0.1"/>
+        </inertial>
+        <visual>
+            <origin xyz="0.0 0.0 0.06" rpy="0.0 0.0 0.0"/>
+            <geometry>
+                <box size="0.256 ${robot_width} ${robot_height}"/>
             </geometry>
             <material name="white"/>
         </visual>
         <collision>
-            <origin xyz="0.0 0.0 0.066" rpy="0.0 0.0 0.0"/>
-            <geometry>
-                <box size="0.256 0.180 0.132" />
+            <origin xyz="0.0 0.0 0.06" rpy="0.0 0.0 0.0"/>
+            <geometry>
+                <box size="0.256 ${robot_width} ${robot_height}"/>
             </geometry>
         </collision>
@@ -45,14 +48,11 @@
     <link name="wheel_left_link">
         <inertial>
-            <mass value="0.1"/>
-            <origin xyz="0 0 0"/>
-            <inertia ixx="0.0001" ixy="0" ixz="0"
-                    iyy="0.0001" iyz="0"
-                    izz="0.0001"/>
-        </inertial>
-        <visual>
-            <origin xyz="0.0 0.0 0.0" rpy="1.5708 0.0 0.0"/>
-            <geometry>
-                <cylinder radius="0.0501" length="0.04"/>
+            <mass value="0.2"/>
+            <inertia ixx="0.1" ixy="0.0" ixz="0.0" iyy="0.1" iyz="0.0" izz="0.2"/>
+        </inertial>
+        <visual>
+            <origin xyz="0.0 0.0 0.0" rpy="1.5708 0.0 0.0"/>
+            <geometry>
+                <cylinder radius="${wheel_radius}" length="${wheel_width}"/>
             </geometry>
             <material name="black"/>
@@ -61,5 +61,5 @@
             <origin xyz="0.0 0.0 0.0" rpy="1.5708 0.0 0.0"/>
             <geometry>
-                <cylinder radius="0.0501" length="0.04"/>
+                <cylinder radius="${wheel_radius}" length="${wheel_width}"/>
             </geometry>
         </collision>
@@ -67,14 +67,11 @@
     <link name="wheel_right_link">
         <inertial>
-            <mass value="0.1"/>
-            <origin xyz="0 0 0"/>
-            <inertia ixx="0.0001" ixy="0" ixz="0"
-                    iyy="0.0001" iyz="0"
-                    izz="0.0001"/>
-        </inertial>
-        <visual>
-            <origin xyz="0.0 0.0 0.0" rpy="1.5708 0.0 0.0"/>
-            <geometry>
-                <cylinder radius="0.0501" length="0.04"/>
+            <mass value="0.2"/>
+            <inertia ixx="0.01" ixy="0.0" ixz="0.0" iyy="0.01" iyz="0.0" izz="0.02"/>
+        </inertial>
+        <visual>
+            <origin xyz="0.0 0.0 0.0" rpy="1.5708 0.0 0.0"/>
+            <geometry>
+                <cylinder radius="${wheel_radius}" length="${wheel_width}"/>
             </geometry>
             <material name="black"/>
@@ -83,28 +80,49 @@
             <origin xyz="0.0 0.0 0.0" rpy="1.5708 0.0 0.0"/>
             <geometry>
-                <cylinder radius="0.0501" length="0.04"/>
-            </geometry>
-        </collision>
-    </link>
-    <link name="caster_wheel">
-        <visual>
-            <origin xyz="0.0 0.0 0.0" rpy="0.0 0.0 0.0"/>
-            <geometry>
-                <sphere radius="0.03"/>
-            </geometry>
-            <material name="black"/>
-        </visual>
-        <collision>
-            <origin xyz="0.0 0.0 0.0" rpy="0.0 0.0 0.0"/>
-            <geometry>
-                <sphere radius="0.03"/>
+                <cylinder radius="${wheel_radius}" length="${wheel_width}"/>
+            </geometry>
+        </collision>
+    </link>
+    <link name="caster_front_link">
+        <inertial>
+            <mass value="0.05"/>
+            <inertia ixx="0.01" ixy="0.0" ixz="0.0" iyy="0.01" iyz="0.0" izz="0.01"/>
+        </inertial>
+        <visual>
+            <origin xyz="0.0 0.0 0.0" rpy="0.0 0.0 0.0"/>
+            <geometry>
+                <sphere radius="${caster_wheel}"/>
+            </geometry>
+        </visual>
+        <collision>
+            <origin xyz="0.0 0.0 0.0" rpy="0.0 0.0 0.0"/>
+            <geometry>
+                <sphere radius="${caster_wheel}"/>
+            </geometry>
+        </collision>
+    </link>
+    <link name="caster_rear_link">
+        <inertial>
+            <mass value="0.05"/>
+            <inertia ixx="0.01" ixy="0.0" ixz="0.0" iyy="0.01" iyz="0.0" izz="0.01"/>
+        </inertial>
+        <visual>
+            <origin xyz="0.0 0.0 0.0" rpy="0.0 0.0 0.0"/>
+            <geometry>
+                <sphere radius="${caster_wheel}"/>
+            </geometry>
+        </visual>
+        <collision>
+            <origin xyz="0.0 0.0 0.0" rpy="0.0 0.0 0.0"/>
+            <geometry>
+                <sphere radius="${caster_wheel}"/>
             </geometry>
         </collision>
     </link>
     <!-- Define the joints -->
-     <joint name="base_joint" type="fixed">
+    <joint name="base_joint" type="fixed">
         <parent link="base_footprint"/>
         <child link="base_link"/>
-        <origin xyz="-0.035 0.0 0.0" rpy="0.0 0.0 0.0"/>
+        <origin xyz="0.0 0.0 ${caster_wheel}" rpy="0.0 0.0 0.0"/>
     </joint>
     <joint name="wheel_right_joint" type="continuous">
@@ -112,5 +130,5 @@
         <child link="wheel_right_link"/>
         <axis xyz="0.0 1.0 0.0"/>
-        <origin xyz="0.035 -0.107 0.018" rpy="0.0 0.0 0.0"/>
+        <origin xyz="0.035 -${wheel_depth/2} 0.02" rpy="0.0 0.0 0.0"/>
     </joint>
     <joint name="wheel_left_joint" type="continuous">
@@ -118,14 +136,19 @@
         <child link="wheel_left_link"/>
         <axis xyz="0.0 1.0 0.0"/>
-        <origin xyz="0.035 0.107 0.018" rpy="0.0 0.0 0.0"/>
-    </joint>
-    <joint name="caster_joint" type="fixed">
-        <parent link="base_link"/>
-        <child link="caster_wheel"/>
-        <!-- <axis xyz="1.0 1.0 0.0"/> -->
-        <origin xyz="-0.098 0.0 0.0" rpy="0.0 0.0 0.0"/>
-    </joint>
-    <!-- Sensors -->
-     <link name="laser_link">
+        <origin xyz="0.035 ${wheel_depth/2} 0.02" rpy="0.0 0.0 0.0"/>
+    </joint>
+    <joint name="caster_front_joint" type="fixed">
+        <parent link="base_link"/>
+        <child link="caster_front_link"/>
+        <axis xyz="0.0 1.0 0.0"/>
+        <origin xyz="-0.08 0.08 -0.01" rpy="0.0 0.0 0.0"/>
+    </joint>
+    <joint name="caster_rear_joint" type="fixed">
+        <parent link="base_link"/>
+        <child link="caster_rear_link"/>
+        <axis xyz="0.0 1.0 0.0"/>
+        <origin xyz="-0.08 -0.08 -0.01" rpy="0.0 0.0 0.0"/>
+    </joint>
+    <link name="laser_link">
     <inertial>
       <origin xyz="-0.011945780406062 -0.000381929217680526 -0.0170649378129477" rpy="0 0 0" />
@@ -167,15 +190,15 @@
         </inertial>
     </link>
-    <joint name="laser_joint" type="fixed">
-        <origin xyz="0.035 0.0 0.142" rpy="0 0 0" />
-        <parent link="base_link" />
-        <child link="laser_link" />
-        <axis xyz="0 0 0" />
-    </joint>
-    <joint name="imu_joint" type="fixed">
-        <origin xyz="-0.0 0.0 0.0" rpy="0 0 0" />
-        <parent link="base_link" />
-        <child link="imu_link" />
-        <axis xyz="0 0 0" />
-    </joint>
+  <joint name="laser_joint" type="fixed">
+    <origin xyz="0.035 0.0 ${robot_height + 0.045}" rpy="0 0 0" />
+    <parent link="base_link" />
+    <child link="laser_link" />
+    <axis xyz="0 0 0" />
+  </joint>
+  <joint name="imu_joint" type="fixed">
+    <origin xyz="-0.0 0.0 0.0" rpy="0 0 0" />
+    <parent link="base_link" />
+    <child link="imu_link" />
+    <axis xyz="0 0 0" />
+  </joint>
 </robot>
