Commit message: 'working code'

File: alphabot_description/urdf/alphabot.urdf.xacro (robot description, xacro)
@@ -111,5 +111,5 @@
         <origin xyz="0.0 0.0 0.04" rpy="0.0 0.0 0.0"/>
     </joint>
-    <joint name="wheel_right_joint" type="continuous">
+    <joint name="right_wheel_joint" type="continuous">
         <parent link="base_link"/>
         <child link="wheel_right_link"/>
@@ -117,5 +117,5 @@
         <origin xyz="0.01 -0.118 0.0" rpy="0.0 0.0 0.0"/>
     </joint>
-    <joint name="wheel_left_joint" type="continuous">
+    <joint name="left_wheel_joint" type="continuous">
         <parent link="base_link"/>
         <child link="wheel_left_link"/>

File: alphabot_description/urdf/alphabot_ros2_control.xacro (robot description, xacro)
@@ -12,5 +12,5 @@
             <hardware>
                 <plugin>alphabot_firmware/AlphabotInterface</plugin>
-                <param name="port">/dev/ttyACM1</param>
+                <param name="port">/dev/ttyACM0</param>
             </hardware>
         </xacro:unless>

Commit message: wheel tracking working functions

File: alphabot_description/urdf/alphabot.urdf.xacro (robot description, xacro)
@@ -111,5 +111,5 @@
         <origin xyz="0.0 0.0 0.04" rpy="0.0 0.0 0.0"/>
     </joint>
-    <joint name="right_wheel_joint" type="continuous">
+    <joint name="wheel_right_joint" type="continuous">
         <parent link="base_link"/>
         <child link="wheel_right_link"/>
@@ -117,5 +117,5 @@
         <origin xyz="0.01 -0.118 0.0" rpy="0.0 0.0 0.0"/>
     </joint>
-    <joint name="left_wheel_joint" type="continuous">
+    <joint name="wheel_left_joint" type="continuous">
         <parent link="base_link"/>
         <child link="wheel_left_link"/>

Commit message: add scanner in description

File: alphabot_description/urdf/alphabot.urdf.xacro (robot description, xacro)
@@ -115,5 +115,5 @@
         <child link="wheel_right_link"/>
         <axis xyz="0.0 1.0 0.0"/>
-        <origin xyz="0.01 -0.118 0.0" rpy="0.0 0.0 0.0"/>
+        <origin xyz="0.062 -0.118 0.0" rpy="0.0 0.0 0.0"/>
     </joint>
     <joint name="wheel_left_joint" type="continuous">
@@ -121,5 +121,5 @@
         <child link="wheel_left_link"/>
         <axis xyz="0.0 1.0 0.0"/>
-        <origin xyz="0.01 0.118 0.0" rpy="0.0 0.0 0.0"/>
+        <origin xyz="0.062 0.118 0.0" rpy="0.0 0.0 0.0"/>
     </joint>
     <joint name="caster_front_joint" type="fixed">
@@ -135,3 +135,30 @@
         <origin xyz="-0.12 0.118 0.0" rpy="0.0 0.0 0.0"/>
     </joint>
+    <link name="laser_link">
+    <inertial>
+      <origin xyz="-0.011945780406062 -0.000381929217680526 -0.0170649378129477" rpy="0 0 0" />
+      <mass value="0.073084435549317" />
+      <inertia ixx="1.96074931730795E-05" ixy="-3.62091076640009E-07" ixz="4.28230084046735E-07"
+               iyy="2.40983835136327E-05" iyz="1.50180909250652E-08"
+               izz="4.14184164228595E-05" />
+    </inertial>
+    <visual>
+      <origin xyz="0 0 0" rpy="0 0 0" />
+      <geometry>
+        <mesh filename="package://alphabot_description/meshes/laser_link.STL" />
+      </geometry>
+    </visual>
+    <collision>
+      <origin xyz="0 0 0" rpy="0 0 0" />
+      <geometry>
+        <mesh filename="package://alphabot_description/meshes/laser_link.STL" />
+      </geometry>
+    </collision>
+  </link>
+  <joint name="laser_joint" type="fixed">
+    <origin xyz="-0.08 0.0 0.16" rpy="0 0 0" />
+    <parent link="base_link" />
+    <child link="laser_link" />
+    <axis xyz="0 0 0" />
+  </joint>
 </robot>

File: alphabot_description/urdf/alphabot_gazebo.xacro (robot description, xacro)
@@ -56,3 +56,38 @@
         </plugin>
     </gazebo>
+    <!-- 2D Laser Sensor -->
+  <gazebo reference="laser_link">
+    <sensor name="lidar" type="ray">
+      <always_on>true</always_on>
+      <visualize>true</visualize>
+      <update_rate>5</update_rate>
+      <ray>
+        <scan>
+          <horizontal>
+            <samples>360</samples>
+            <resolution>1.00000</resolution>
+            <min_angle>0.000000</min_angle>
+            <max_angle>6.280000</max_angle>
+          </horizontal>
+        </scan>
+        <range>
+          <min>0.120000</min>
+          <max>12.0</max>
+          <resolution>0.02</resolution>
+        </range>
+        <noise>
+          <type>gaussian</type>
+          <mean>0.0</mean>
+          <stddev>0.01</stddev>
+        </noise>
+      </ray>
+      <plugin name="scan" filename="libgazebo_ros_ray_sensor.so">
+        <ros>
+          <remapping>~/out:=scan</remapping>
+        </ros>
+        <output_type>sensor_msgs/LaserScan</output_type>
+        <frame_name>laser_link</frame_name>
+      </plugin>
+    </sensor>
+  </gazebo>
 </robot>

Commit message: add imu in urdf and gazebo, create launch file to use cartographer

File: alphabot_description/urdf/alphabot.urdf.xacro (robot description, xacro)
@@ -156,4 +156,23 @@
     </collision>
   </link>
+  <link name="imu_link">
+        <collision>
+            <origin xyz="0 0 0" rpy="0 0 0"/>
+            <geometry>
+                <box size="0.005 0.005 0.005"/>
+            </geometry>
+        </collision>
+        <visual>
+            <origin xyz="0 0 0" rpy="0 0 0"/>
+            <geometry>
+                <box size="0.005 0.005 0.005"/>
+            </geometry>
+        </visual>
+        <inertial>
+            <mass value="0.001" />
+            <origin xyz="0 0 0" rpy="0 0 0"/>
+            <inertia ixx="0.00000015" ixy="0" ixz="0" iyy="0.00000015" iyz="0" izz="0.00000015" />
+        </inertial>
+    </link>
   <joint name="laser_joint" type="fixed">
     <origin xyz="-0.08 0.0 0.16" rpy="0 0 0" />
@@ -162,3 +181,9 @@
     <axis xyz="0 0 0" />
   </joint>
+  <joint name="imu_joint" type="fixed">
+    <origin xyz="-0.0 0.0 0.0" rpy="0 0 0" />
+    <parent link="base_link" />
+    <child link="imu_link" />
+    <axis xyz="0 0 0" />
+  </joint>
 </robot>

File: alphabot_description/urdf/alphabot_gazebo.xacro (robot description, xacro)
@@ -91,3 +91,53 @@
     </sensor>
   </gazebo>
+  <!-- IMU SENSOR -->
+   <gazebo reference="imu_link">
+    <sensor name="imu" type="imu">
+        <always_on>true</always_on>
+        <update_rate>100</update_rate>
+        <imu>
+          <angular_velocity>
+            <x>
+              <noise type="gaussian">
+                <mean>0.0</mean>
+                <stddev>2e-4</stddev>
+              </noise>
+            </x>
+            <y>
+              <noise type="gaussian">
+                <mean>0.0</mean>
+                <stddev>2e-4</stddev>
+              </noise>
+            </y>
+            <z>
+              <noise type="gaussian">
+                <mean>0.0</mean>
+                <stddev>2e-4</stddev>
+              </noise>
+            </z>
+          </angular_velocity>
+          <linear_acceleration>
+            <x>
+              <noise type="gaussian">
+                <mean>0.0</mean>
+                <stddev>1.7e-2</stddev>
+              </noise>
+            </x>
+            <y>
+              <noise type="gaussian">
+                <mean>0.0</mean>
+                <stddev>1.7e-2</stddev>
+              </noise>
+            </y>
+            <z>
+              <noise type="gaussian">
+                <mean>0.0</mean>
+                <stddev>1.7e-2</stddev>
+              </noise>
+            </z>
+          </linear_acceleration>
+        </imu>
+        <plugin name="imu" filename="libgazebo_ros_imu_sensor.so"/>
+    </sensor>
+  </gazebo>
 </robot>

Commit message: create new launch file in alphabot_mapping to run slam with the config file. modified simulation.launch.py to run all functionality for slam or amcl

File: alphabot_description/urdf/alphabot.urdf.xacro (robot description, xacro)
@@ -46,5 +46,5 @@
             <origin xyz="0.0 0.0 0.0" rpy="1.5708 0.0 0.0"/>
             <geometry>
-                <cylinder radius="0.03" length="0.025"/>
+                <cylinder radius="0.035" length="0.025"/>
             </geometry>
         </collision>
@@ -58,5 +58,5 @@
             <origin xyz="0.0 0.0 0.0" rpy="1.5708 0.0 0.0"/>
             <geometry>
-                <cylinder radius="0.03" length="0.025"/>
+                <cylinder radius="0.035" length="0.025"/>
             </geometry>
             <material name="black"/>
@@ -65,5 +65,5 @@
             <origin xyz="0.0 0.0 0.0" rpy="1.5708 0.0 0.0"/>
             <geometry>
-                <cylinder radius="0.03" length="0.025"/>
+                <cylinder radius="0.035" length="0.025"/>
             </geometry>
         </collision>

Commit message: update urdf to new robot

File: alphabot_description/urdf/alphabot.urdf.xacro (robot description, xacro)
@@ -5,4 +5,10 @@
     <xacro:include filename="$(find alphabot_description)/urdf/alphabot_gazebo.xacro"/>
     <xacro:include filename="$(find alphabot_description)/urdf/alphabot_ros2_control.xacro"/>
+    <xacro:property name="wheel_radius" value="0.034" />
+    <xacro:property name="wheel_width" value="0.012" />
+    <xacro:property name="robot_height" value="0.116" />
+    <xacro:property name="robot_width" value="0.256" />
+    <xacro:property name="wheel_depth" value="0.256" />
+    <xacro:property name="caster_wheel" value="0.01468" />
     <material name="white">
         <color rgba="1 1 1 1"/>
@@ -14,5 +20,5 @@
     <link name="base_link">
         <inertial>
-            <mass value="1.5"/>
+            <mass value="2.0"/>
             <inertia ixx="0.1" ixy="0.0" ixz="0.0" iyy="0.1" iyz="0.0" izz="0.1"/>
         </inertial>
@@ -20,5 +26,5 @@
             <origin xyz="0.0 0.0 0.06" rpy="0.0 0.0 0.0"/>
             <geometry>
-                <box size="0.33 0.33 0.15"/>
+                <box size="0.256 0.256 0.116"/>
             </geometry>
             <material name="white"/>
@@ -27,5 +33,5 @@
             <origin xyz="0.0 0.0 0.15" rpy="0.0 0.0 0.0"/>
             <geometry>
-                <box size="0.33 0.33 0.0"/>
+                <box size="0.256 0.256 0.116"/>
             </geometry>
         </collision>
@@ -39,5 +45,5 @@
             <origin xyz="0.0 0.0 0.0" rpy="1.5708 0.0 0.0"/>
             <geometry>
-                <cylinder radius="0.035" length="0.025"/>
+                <cylinder radius="${wheel_radius}" length="${wheel_width}"/>
             </geometry>
             <material name="black"/>
@@ -46,5 +52,5 @@
             <origin xyz="0.0 0.0 0.0" rpy="1.5708 0.0 0.0"/>
             <geometry>
-                <cylinder radius="0.035" length="0.025"/>
+                <cylinder radius="${wheel_radius}" length="${wheel_width}"/>
             </geometry>
         </collision>
@@ -58,5 +64,5 @@
             <origin xyz="0.0 0.0 0.0" rpy="1.5708 0.0 0.0"/>
             <geometry>
-                <cylinder radius="0.035" length="0.025"/>
+                <cylinder radius="${wheel_radius}" length="${wheel_width}"/>
             </geometry>
             <material name="black"/>
@@ -65,5 +71,5 @@
             <origin xyz="0.0 0.0 0.0" rpy="1.5708 0.0 0.0"/>
             <geometry>
-                <cylinder radius="0.035" length="0.025"/>
+                <cylinder radius="${wheel_radius}" length="${wheel_width}"/>
             </geometry>
         </collision>
@@ -77,5 +83,5 @@
             <origin xyz="0.0 0.0 0.0" rpy="0.0 0.0 0.0"/>
             <geometry>
-                <sphere radius="0.03"/>
+                <sphere radius="${caster_wheel}"/>
             </geometry>
         </visual>
@@ -83,5 +89,5 @@
             <origin xyz="0.0 0.0 0.0" rpy="0.0 0.0 0.0"/>
             <geometry>
-                <sphere radius="0.03"/>
+                <sphere radius="${caster_wheel}"/>
             </geometry>
         </collision>
@@ -95,5 +101,5 @@
             <origin xyz="0.0 0.0 0.0" rpy="0.0 0.0 0.0"/>
             <geometry>
-                <sphere radius="0.035"/>
+                <sphere radius="${caster_wheel}"/>
             </geometry>
         </visual>
@@ -101,5 +107,5 @@
             <origin xyz="0.0 0.0 0.0" rpy="0.0 0.0 0.0"/>
             <geometry>
-                <sphere radius="0.03"/>
+                <sphere radius="${caster_wheel}"/>
             </geometry>
         </collision>
@@ -109,5 +115,5 @@
         <parent link="base_footprint"/>
         <child link="base_link"/>
-        <origin xyz="0.0 0.0 0.04" rpy="0.0 0.0 0.0"/>
+        <origin xyz="0.0 0.0 ${caster_wheel}" rpy="0.0 0.0 0.0"/>
     </joint>
     <joint name="wheel_right_joint" type="continuous">
@@ -115,5 +121,5 @@
         <child link="wheel_right_link"/>
         <axis xyz="0.0 1.0 0.0"/>
-        <origin xyz="0.062 -0.118 0.0" rpy="0.0 0.0 0.0"/>
+        <origin xyz="0.060 -0.105 0.02" rpy="0.0 0.0 0.0"/>
     </joint>
     <joint name="wheel_left_joint" type="continuous">
@@ -121,5 +127,5 @@
         <child link="wheel_left_link"/>
         <axis xyz="0.0 1.0 0.0"/>
-        <origin xyz="0.062 0.118 0.0" rpy="0.0 0.0 0.0"/>
+        <origin xyz="0.060 0.105 0.02" rpy="0.0 0.0 0.0"/>
     </joint>
     <joint name="caster_front_joint" type="fixed">
@@ -127,5 +133,5 @@
         <child link="caster_front_link"/>
         <axis xyz="0.0 1.0 0.0"/>
-        <origin xyz="-0.12 -0.118 0.0" rpy="0.0 0.0 0.0"/>
+        <origin xyz="-0.08 -0.08 0.0" rpy="0.0 0.0 0.0"/>
     </joint>
     <joint name="caster_rear_joint" type="fixed">
@@ -133,5 +139,5 @@
         <child link="caster_rear_link"/>
         <axis xyz="0.0 1.0 0.0"/>
-        <origin xyz="-0.12 0.118 0.0" rpy="0.0 0.0 0.0"/>
+        <origin xyz="-0.08 0.08 0.0" rpy="0.0 0.0 0.0"/>
     </joint>
     <link name="laser_link">
@@ -176,5 +182,5 @@
     </link>
   <joint name="laser_joint" type="fixed">
-    <origin xyz="-0.08 0.0 0.16" rpy="0 0 0" />
+    <origin xyz="-0.065 0.0 ${robot_height + 0.005}" rpy="0 0 0" />
     <parent link="base_link" />
     <child link="laser_link" />

File: alphabot_description/urdf/alphabot_ros2_control.xacro (robot description, xacro)
@@ -56,6 +56,6 @@
         <joint name="wheel_right_joint">
             <command_interface name="velocity">
-              <param name="min">-0.35</param>
-              <param name="max">0.35</param>
+              <param name="min">-0.5</param>
+              <param name="max">0.5</param>
             </command_interface>
             <state_interface name="position" />
@@ -64,6 +64,6 @@
         <joint name="wheel_left_joint">
             <command_interface name="velocity">
-              <param name="min">-0.35</param>
-              <param name="max">0.35</param>
+              <param name="min">-0.5</param>
+              <param name="max">0.5</param>
             </command_interface>
             <state_interface name="position" />

Commit message: modify alphabot_description to work with gazebo harmonic

File: alphabot_description/urdf/alphabot.urdf.xacro (robot description, xacro)
@@ -1,9 +1,11 @@
 <?xml version="1.0"?>
 <robot xmlns:xacro="http://www.ros.org/wiki/xacro" name="alphabot">
+    <!-- Start GZ or Ignition depending on ROS 2 Version -->
+    <xacro:arg name="is_ignition" default="true"/>
     <!-- Load Simulated or Real Hardware Interfaces -->
     <xacro:arg name="is_sim" default="true"/>
     <xacro:include filename="$(find alphabot_description)/urdf/alphabot_gazebo.xacro"/>
     <xacro:include filename="$(find alphabot_description)/urdf/alphabot_ros2_control.xacro"/>
-    <xacro:include filename="$(find alphabot_description)/urdf/depth_camera.xacro" />
+    <!-- <xacro:include filename="$(find alphabot_description)/urdf/depth_camera.xacro" /> -->
     <xacro:property name="wheel_radius" value="0.034" />
     <xacro:property name="wheel_width" value="0.012" />
@@ -17,4 +19,10 @@
     <material name="black">
         <color rgba="0 0 0 1"/>
+    </material>
+    <material name="silver">
+        <color rgba="0.79 0.82 0.93 1"/>
+    </material>
+    <material name="dark_grey">
+        <color rgba="0.3 0.3 0.3 1"/>
     </material>
     <link name="base_footprint"/>

File: alphabot_description/urdf/alphabot_gazebo.xacro (robot description, xacro)
@@ -50,11 +50,22 @@
     </gazebo>
     <gazebo>
-        <plugin filename="libgazebo_ros2_control.so" name="gazebo_ros2_control">
-            <robot_param>robot_description</robot_param>
-            <robot_param_node>robot_state_publisher</robot_param_node>
-            <parameters>$(find alphabot_controller)/config/alphabot_controllers.yaml</parameters>
-        </plugin>
-    </gazebo>
-    <!-- 2D Laser Sensor -->
+    <!-- ROS 2 Humble -->
+    <xacro:if value="$(arg is_ignition)">
+      <plugin filename="ign_ros2_control-system" name="ign_ros2_control::IgnitionROS2ControlPlugin">
+        <parameters>$(find alphabot_controller)/config/alphabot_controllers.yaml</parameters>
+      </plugin>
+      <plugin filename="ignition-gazebo-imu-system" name="ignition::gazebo::systems::Imu">
+      </plugin>
+    </xacro:if>
+    <!-- ROS 2 Iron or above -->
+    <xacro:unless value="$(arg is_ignition)">
+      <plugin filename="gz_ros2_control-system" name="gz_ros2_control::GazeboSimROS2ControlPlugin">
+        <parameters>$(find alphabot_controller)/config/alphabot_controllers.yaml</parameters>
+      </plugin>
+      <plugin filename="gz-sim-imu-system" name="gz::sim::systems::Imu">
+      </plugin>
+    </xacro:unless>
+  </gazebo>
+<!--
   <gazebo reference="laser_link">
     <sensor name="lidar" type="ray">
@@ -91,5 +102,4 @@
     </sensor>
   </gazebo>
-  <!-- IMU SENSOR -->
    <gazebo reference="imu_link">
     <sensor name="imu" type="imu">
@@ -140,4 +150,4 @@
         <plugin name="imu" filename="libgazebo_ros_imu_sensor.so"/>
     </sensor>
-  </gazebo>
+  </gazebo> -->
 </robot>

File: alphabot_description/urdf/camera.xacro (robot description, xacro)
@@ -1,7 +1,4 @@
 <?xml version="1.0"?>
 <robot xmlns:xacro="http://www.ros.org/wiki/xacro" >
-    <material name="red">
-        <color rgba="1 0 0 1"/>
-    </material>
     <joint name="camera_joint" type="fixed">
         <parent link="base_link"/>
@@ -14,5 +11,7 @@
                 <box size="0.010 0.03 0.03"/>
             </geometry>
-            <material name="red"/>
+            <material>
+                <color rgba="1 0 0 1"/>
+            </material>
         </visual>
     </link>

Commit message: Working with imu

File: alphabot_description/urdf/alphabot.urdf.xacro (robot description, xacro)
@@ -189,5 +189,5 @@
   </joint>
   <joint name="imu_joint" type="fixed">
-    <origin xyz="-0.0 0.0 0.0" rpy="0 0 0" />
+    <origin xyz="-0.0 0.0 0.05" rpy="0 0 0" />
     <parent link="base_link" />
     <child link="imu_link" />

Commit message: working code

File: alphabot_description/urdf/alphabot.urdf.xacro (robot description, xacro)
@@ -161,5 +161,5 @@
       <origin xyz="0 0 0" rpy="0 0 0" />
       <geometry>
-        <mesh filename="package://alphabot_description/meshes/laser_link.STL" />
+        <box size="0.08 0.08 0.03" />
       </geometry>
     </visual>
@@ -167,5 +167,5 @@
       <origin xyz="0 0 0" rpy="0 0 0" />
       <geometry>
-        <mesh filename="package://alphabot_description/meshes/laser_link.STL" />
+        <box size="0.08 0.08 0.03" />
       </geometry>
     </collision>

Commit message: update the description

File: alphabot_description/urdf/alphabot.urdf.xacro (robot description, xacro)
@@ -8,10 +8,10 @@
     <xacro:include filename="$(find alphabot_description)/urdf/alphabot_ros2_control.xacro"/>
     <!-- <xacro:include filename="$(find alphabot_description)/urdf/depth_camera.xacro" /> -->
-    <xacro:property name="wheel_radius" value="0.034" />
-    <xacro:property name="wheel_width" value="0.012" />
-    <xacro:property name="robot_height" value="0.116" />
-    <xacro:property name="robot_width" value="0.256" />
-    <xacro:property name="wheel_depth" value="0.256" />
-    <xacro:property name="caster_wheel" value="0.01468" />
+    <xacro:property name="wheel_radius" value="0.051" />
+    <xacro:property name="wheel_width" value="0.040" />
+    <xacro:property name="robot_height" value="0.093" />
+    <xacro:property name="robot_width" value="0.20" />
+    <xacro:property name="wheel_depth" value="0.22" />
+    <xacro:property name="caster_wheel" value="0.018" />
     <material name="white">
         <color rgba="1 1 1 1"/>
@@ -35,5 +35,5 @@
             <origin xyz="0.0 0.0 0.06" rpy="0.0 0.0 0.0"/>
             <geometry>
-                <box size="0.256 0.256 0.116"/>
+                <box size="0.256 0.256 ${robot_height}"/>
             </geometry>
             <material name="white"/>
@@ -42,5 +42,5 @@
             <origin xyz="0.0 0.0 0.15" rpy="0.0 0.0 0.0"/>
             <geometry>
-                <box size="0.256 0.256 0.116"/>
+                <box size="0.256 0.256 ${robot_height}"/>
             </geometry>
         </collision>
@@ -102,5 +102,5 @@
         </collision>
     </link>
-    <link name="caster_rear_link">
+    <!-- <link name="caster_rear_link">
         <inertial>
             <mass value="0.05"/>
@@ -119,5 +119,5 @@
             </geometry>
         </collision>
-    </link>
+    </link> -->
     <!-- Define the joints -->
     <joint name="base_joint" type="fixed">
@@ -130,5 +130,5 @@
         <child link="wheel_right_link"/>
         <axis xyz="0.0 1.0 0.0"/>
-        <origin xyz="0.060 -0.105 0.02" rpy="0.0 0.0 0.0"/>
+        <origin xyz="0.035 -${wheel_depth/2} 0.02" rpy="0.0 0.0 0.0"/>
     </joint>
     <joint name="wheel_left_joint" type="continuous">
@@ -136,5 +136,5 @@
         <child link="wheel_left_link"/>
         <axis xyz="0.0 1.0 0.0"/>
-        <origin xyz="0.060 0.105 0.02" rpy="0.0 0.0 0.0"/>
+        <origin xyz="0.035 ${wheel_depth/2} 0.02" rpy="0.0 0.0 0.0"/>
     </joint>
     <joint name="caster_front_joint" type="fixed">
@@ -142,12 +142,12 @@
         <child link="caster_front_link"/>
         <axis xyz="0.0 1.0 0.0"/>
-        <origin xyz="-0.08 -0.08 0.0" rpy="0.0 0.0 0.0"/>
-    </joint>
-    <joint name="caster_rear_joint" type="fixed">
+        <origin xyz="-0.08 0.0 0.0" rpy="0.0 0.0 0.0"/>
+    </joint>
+    <!-- <joint name="caster_rear_joint" type="fixed">
         <parent link="base_link"/>
         <child link="caster_rear_link"/>
         <axis xyz="0.0 1.0 0.0"/>
         <origin xyz="-0.08 0.08 0.0" rpy="0.0 0.0 0.0"/>
-    </joint>
+    </joint> -->
     <link name="laser_link">
     <inertial>
@@ -191,5 +191,5 @@
     </link>
   <joint name="laser_joint" type="fixed">
-    <origin xyz="-0.065 0.0 ${robot_height + 0.005}" rpy="0 0 0" />
+    <origin xyz="0.035 0.0 ${robot_height + 0.005 + 0.015}" rpy="0 0 0" />
     <parent link="base_link" />
     <child link="laser_link" />
