Commit message: Creating alphabot_navigation pkg and costmap

File: alphabot_description/urdf/alphabot.urdf.xacro (robot description, xacro)
@@ -191,5 +191,5 @@
     </link>
   <joint name="laser_joint" type="fixed">
-    <origin xyz="0.035 0.0 ${robot_height + 0.005 + 0.015}" rpy="0 0 0" />
+    <origin xyz="0.035 0.0 ${robot_height + 0.005 + 0.02}" rpy="0 0 0" />
     <parent link="base_link" />
     <child link="laser_link" />

File: alphabot_description/urdf/alphabot_gazebo.xacro (robot description, xacro)
@@ -115,6 +115,6 @@
         </scan>
         <range>
-          <min>0.120000</min>
-          <max>12.0</max>
+          <min>0.20000</min>
+          <max>6.0</max>
           <resolution>0.02</resolution>
         </range>

Commit message: fixed motion plugin

File: alphabot_description/urdf/alphabot.urdf.xacro (robot description, xacro)
@@ -191,5 +191,5 @@
     </link>
   <joint name="laser_joint" type="fixed">
-    <origin xyz="0.035 0.0 ${robot_height + 0.005 + 0.02}" rpy="0 0 0" />
+    <origin xyz="0.035 0.0 ${robot_height + 0.005 + 0.04}" rpy="0 0 0" />
     <parent link="base_link" />
     <child link="laser_link" />

Commit message: vreate behavior

File: alphabot_description/urdf/alphabot.urdf.xacro (robot description, xacro)
@@ -40,5 +40,5 @@
         </visual>
         <collision>
-            <origin xyz="0.0 0.0 0.15" rpy="0.0 0.0 0.0"/>
+            <origin xyz="0.0 0.0 0.06" rpy="0.0 0.0 0.0"/>
             <geometry>
                 <box size="0.256 0.256 ${robot_height}"/>
@@ -191,5 +191,5 @@
     </link>
   <joint name="laser_joint" type="fixed">
-    <origin xyz="0.035 0.0 ${robot_height + 0.005 + 0.04}" rpy="0 0 0" />
+    <origin xyz="0.035 0.0 ${robot_height + 0.045}" rpy="0 0 0" />
     <parent link="base_link" />
     <child link="laser_link" />

File: alphabot_description/urdf/alphabot_gazebo.xacro (robot description, xacro)
@@ -110,6 +110,6 @@
             <samples>360</samples>
             <resolution>1.00000</resolution>
-            <min_angle>0.000000</min_angle>
-            <max_angle>6.280000</max_angle>
+            <min_angle>-1.57</min_angle>
+            <max_angle>1.57</max_angle>
           </horizontal>
         </scan>

Commit message: update parameters

File: alphabot_description/urdf/alphabot.urdf.xacro (robot description, xacro)
@@ -35,5 +35,5 @@
             <origin xyz="0.0 0.0 0.06" rpy="0.0 0.0 0.0"/>
             <geometry>
-                <box size="0.256 0.256 ${robot_height}"/>
+                <box size="0.256 ${robot_width} ${robot_height}"/>
             </geometry>
             <material name="white"/>
@@ -42,5 +42,5 @@
             <origin xyz="0.0 0.0 0.06" rpy="0.0 0.0 0.0"/>
             <geometry>
-                <box size="0.256 0.256 ${robot_height}"/>
+                <box size="0.256 ${robot_width} ${robot_height}"/>
             </geometry>
         </collision>
@@ -102,5 +102,5 @@
         </collision>
     </link>
-    <!-- <link name="caster_rear_link">
+    <link name="caster_rear_link">
         <inertial>
             <mass value="0.05"/>
@@ -119,5 +119,5 @@
             </geometry>
         </collision>
-    </link> -->
+    </link>
     <!-- Define the joints -->
     <joint name="base_joint" type="fixed">
@@ -142,12 +142,12 @@
         <child link="caster_front_link"/>
         <axis xyz="0.0 1.0 0.0"/>
-        <origin xyz="-0.08 0.0 0.0" rpy="0.0 0.0 0.0"/>
-    </joint>
-    <!-- <joint name="caster_rear_joint" type="fixed">
+        <origin xyz="-0.08 0.08 -0.01" rpy="0.0 0.0 0.0"/>
+    </joint>
+    <joint name="caster_rear_joint" type="fixed">
         <parent link="base_link"/>
         <child link="caster_rear_link"/>
         <axis xyz="0.0 1.0 0.0"/>
-        <origin xyz="-0.08 0.08 0.0" rpy="0.0 0.0 0.0"/>
-    </joint> -->
+        <origin xyz="-0.08 -0.08 -0.01" rpy="0.0 0.0 0.0"/>
+    </joint>
     <link name="laser_link">
     <inertial>

Commit message: add camera link and add gz_image_bridge

File: alphabot_description/urdf/alphabot.urdf.xacro (robot description, xacro)
@@ -7,4 +7,5 @@
     <xacro:include filename="$(find alphabot_description)/urdf/alphabot_gazebo.xacro"/>
     <xacro:include filename="$(find alphabot_description)/urdf/alphabot_ros2_control.xacro"/>
+    <xacro:include filename="$(find alphabot_description)/urdf/camera.xacro" />
     <!-- <xacro:include filename="$(find alphabot_description)/urdf/depth_camera.xacro" /> -->
     <material name="white">

File: alphabot_description/urdf/camera.xacro (robot description, xacro)
@@ -1,8 +1,8 @@
 <?xml version="1.0"?>
-<robot xmlns:xacro="http://www.ros.org/wiki/xacro" >
+<robot xmlns:xacro="http://www.ros.org/wiki/xacro">
     <joint name="camera_joint" type="fixed">
         <parent link="base_link"/>
         <child link="camera_link"/>
-        <origin xyz="0.128 0 0.095" rpy="0 0 0"/>
+        <origin xyz="0.128 0 0.1" rpy="0 0 0"/>
     </joint>
     <link name="camera_link">
@@ -11,7 +11,5 @@
                 <box size="0.010 0.03 0.03"/>
             </geometry>
-            <material>
-                <color rgba="1 0 0 1"/>
-            </material>
+            <material name="red"/>
         </visual>
     </link>
@@ -19,13 +17,14 @@
         <parent link="camera_link"/>
         <child link="camera_link_optical"/>
-        <origin xyz="0 0 0" rpy="${-pi/2} 0 ${-pi/2}"/>
+        <origin xyz="0 0 0" rpy="${-3.14/2} 0 ${-3.14/2}"/>
     </joint>
-    <link name="camera_link_optical"></link>
+    <link name="camera_link_optical"/>
     <gazebo reference="camera_link">
         <material>Gazebo/Red</material>
         <sensor name="camera" type="camera">
-            <pose> 0 0 0 0 0 0 </pose>
+            <pose>0 0 0 0 0 0</pose>
             <visualize>true</visualize>
             <update_rate>10</update_rate>
+            <!-- <topic>/camera</topic> -->
             <camera>
                 <horizontal_fov>1.089</horizontal_fov>
@@ -40,5 +39,8 @@
                 </clip>
             </camera>
-            <plugin name="camera_controller" filename="libgazebo_ros_camera.so">
+            <plugin name="camera_controller" filename="libgazebo_ros_camera_system.so">
+                <ros>
+                    <namespace>/</namespace>
+                </ros>
                 <frame_name>camera_link_optical</frame_name>
             </plugin>

Commit message: add different backend for slam

File: alphabot_description/urdf/alphabot.urdf.xacro (robot description, xacro)
@@ -20,4 +20,7 @@
     <material name="dark_grey">
         <color rgba="0.3 0.3 0.3 1"/>
+    </material>
+    <material name="red">
+        <color rgba="1 0 0 1"/>
     </material>
     <link name="base_footprint"/>
