Commit message: fixing scanner and wheel directions

File: alphabot_description/urdf/servicebot/robot.urdf.xacro (robot description, xacro)
@@ -247,5 +247,5 @@
   <parent link="base_link"/>
   <child link="wheel_left_link"/>
-  <axis xyz="0.0 -1.0 0.0"/>
+  <axis xyz="0.0 1.0 0.0"/>
 </joint>
 <joint name="wheel_right_joint" type="continuous">
@@ -253,5 +253,5 @@
   <parent link="base_link"/>
   <child link="wheel_right_link"/>
-  <axis xyz="0.0 -1.0 0.0"/>
+  <axis xyz="0.0 1.0 0.0"/>
 </joint>
 <joint name="laser_joint" type="fixed">
